File: griffin.sch (KiCad schematic (older format))
At the start: 0 parts

Commit message: update
Parts:
- added C? (x5): C, symbol Device:C
- added D?: LED, symbol Device:LED
- added F?: Fuse, symbol Device:Fuse
- added J? (x4): Conn_01x08_Female, symbol Connector:Conn_01x08_Female
- added J?: USB_B_Micro, symbol Connector:USB_B_Micro
- added R?: R, symbol Device:R
- added U?: CH340C, Package_SO:SOIC-16_3.9x9.9mm_P1.27mm, symbol Interface_USB:CH340C
- added U?: STC89C52RC-40I, lc_lib:LQFP-44_10X10X08P, symbol lc_MCU:STC89C52RC-40I
- added Y?: Crystal, symbol Device:Crystal
Connections:
- net labels added: +5V, DM, DP, GND, RST
- wire segments 0 -> 74

Commit message: schematic for STM32F103C8T6
Parts:
- removed C? (x5): C, symbol Device:C
- removed D?: LED, symbol Device:LED
- removed F?: Fuse, symbol Device:Fuse
- removed J? (x4): Conn_01x08_Female, symbol Connector:Conn_01x08_Female
- removed J?: USB_B_Micro, symbol Connector:USB_B_Micro
- removed R?: R, symbol Device:R
- removed U?: CH340C, Package_SO:SOIC-16_3.9x9.9mm_P1.27mm, symbol Interface_USB:CH340C
- removed U?: STC89C52RC-40I, lc_lib:LQFP-44_10X10X08P, symbol lc_MCU:STC89C52RC-40I
- removed Y?: Crystal, symbol Device:Crystal
- added C1, C11, C12, C13, C14, C2, C5, C6, C9: 104, symbol Device:C
- added C10: 105, symbol Device:C
- added C3, C4: 15pF, symbol Device:C
- added C7, C8: 22pF, symbol Device:C
- added D1, D2: LED, symbol Device:LED
- added F1: Fuse 0.75A, symbol Device:Fuse
- added IC1: ME6211C33M5G-N, SOT95P270X145-5N, symbol ME6211C33M5G-N:ME6211C33M5G-N
- added J1: USB_B_Micro, symbol Connector:USB_B_Micro
- added J2: Conn_02x03_Odd_Even, symbol Connector_Generic:Conn_02x03_Odd_Even
- added J3, J5: Conn_01x04, symbol Connector_Generic:Conn_01x04
- added J4: Conn_01x11, symbol Connector_Generic:Conn_01x11
- added J6, J7: Conn_01x20, symbol Connector_Generic:Conn_01x20
- added J8: Conn_01x14, symbol Connector_Generic:Conn_01x14
- added J9: Conn_01x08, symbol Connector_Generic:Conn_01x08
- added R1: 1M, symbol Device:R
- added R2, R8, R9: 10k, symbol Device:R
- added R3, R4: 10R, symbol Device:R
- added R5: 1.5k, symbol Device:R
- added R6, R7: 1k, symbol Device:R
- added SW1, SW2: SW_Push, symbol Switch:SW_Push
- added U1: STM32F103C8T6, lc_lib:LQFP-48_7X7X05P, symbol lc_MCU:STM32F103C8T6
- added U2, U3: CA56-12EWA, Display_7Segment:CA56-12EWA, symbol Display_Character:CA56-12EWA
- added U4: TM1640_[C41327], lc_lib:SOP-28_300MIL, symbol lc_IC:TM1640_[C41327]
- added Y1: 32.768KHz, symbol Device:Crystal
- added Y2: 8MHz, symbol Device:Crystal
Connections:
- net labels added: +3.3V, BOOT0, BOOT1, KEY0, RESET, SWCLK, SWDAT, USB_D+, USB_D-, VBAT
- net labels removed: DM, DP, RST
- wire segments 74 -> 132
Other:
- note added: "Battery"
- note added: "Boot mode selection"
- note added: "DC DC Convertor"
- note added: "IO Connector"
- note added: "Key"
- note added: "LCD Connector"
- note added: "LED\n\n"
- note added: "Reset\n"
- note added: "STM32F103C8T6\n"
- note added: "SWD\n"
- note added: "USB\n"

Commit message: update
Parts:
- removed U2, U3: CA56-12EWA, Display_7Segment:CA56-12EWA, symbol Display_Character:CA56-12EWA
- removed U4: TM1640_[C41327], lc_lib:SOP-28_300MIL, symbol lc_IC:TM1640_[C41327]
- C1, C10, C11, C12, C13, C14, C2, C3, C4, C5, C6, C7, C8, C9: footprint (none) -> Capacitor_SMD:C_0603_1608Metric
- D1, D2: footprint (none) -> LED_SMD:LED_0603_1608Metric
- F1: footprint (none) -> Fuse:Fuse_0805_2012Metric
- IC1: footprint SOT95P270X145-5N -> (none)
- J1: footprint (none) -> Connector_USB:USB_Micro-AB_Molex_47590-0001
- J2: footprint (none) -> Connector_PinHeader_2.54mm:PinHeader_1x06_P2.54mm_Vertical
- J3, J5: footprint (none) -> Connector_PinHeader_2.54mm:PinHeader_1x04_P2.54mm_Vertical
- J4: footprint (none) -> Connector_PinHeader_2.54mm:PinHeader_1x11_P2.54mm_Vertical
- J6, J7: footprint (none) -> Connector_PinHeader_2.54mm:PinHeader_1x20_P2.54mm_Vertical
- J8: footprint (none) -> Connector_PinHeader_2.54mm:PinHeader_1x14_P2.54mm_Vertical
- J9: footprint (none) -> Connector_PinHeader_2.54mm:PinHeader_1x08_P2.54mm_Vertical
- R1, R2, R3, R4, R5, R6, R7, R8, R9: footprint (none) -> Resistor_SMD:R_0603_1608Metric
- SW1: footprint (none) -> Button_Switch_THT:SW_MEC_5GTH9
- SW2: footprint (none) -> Button_Switch_THT:SW_PUSH_6mm
- Y1, Y2: footprint (none) -> Crystal:Crystal_Round_D3.0mm_Vertical

Commit message: update
Parts:
- removed U1: STM32F103C8T6, lc_lib:LQFP-48_7X7X05P, symbol lc_MCU:STM32F103C8T6
- added U1: STM32F103C8Tx, Package_QFP:LQFP-48_7x7mm_P0.5mm, symbol MCU_ST_STM32F1:STM32F103C8Tx
- IC1: footprint (none) -> griffin:SOT95P270X145-5N
- J2: footprint Connector_PinHeader_2.54mm:PinHeader_1x06_P2.54mm_Vertical -> Connector_PinSocket_2.54mm:PinSocket_1x06_P2.54mm_Vertical
- J3, J5: footprint Connector_PinHeader_2.54mm:PinHeader_1x04_P2.54mm_Vertical -> Connector_PinSocket_2.54mm:PinSocket_1x04_P2.54mm_Vertical
- J4: footprint Connector_PinHeader_2.54mm:PinHeader_1x11_P2.54mm_Vertical -> Connector_PinSocket_2.54mm:PinSocket_1x11_P2.54mm_Vertical
- J8: footprint Connector_PinHeader_2.54mm:PinHeader_1x14_P2.54mm_Vertical -> Connector_PinSocket_2.54mm:PinSocket_1x14_P2.54mm_Vertical
- J9: footprint Connector_PinHeader_2.54mm:PinHeader_1x08_P2.54mm_Vertical -> Connector_PinSocket_2.54mm:PinSocket_1x08_P2.54mm_Vertical
- Y2: footprint Crystal:Crystal_Round_D3.0mm_Vertical -> Crystal:Crystal_HC49-U_Vertical
Connections:
- net USB_D+ is gone; now on net PA12: R4.1
- net USB_D- is gone; now on net PA11: R5.1
- net +3V3: now also J5.1 (Pin_1), J6.3 (Pin_3), J7.1 (Pin_1), J9.2 (Pin_2), U1.24 (VDD), U1.36 (VDD), U1.48 (VDD), U1.9 (VDDA)
- net +5V: now also J4.1 (Pin_1), J6.2 (Pin_2), J7.2 (Pin_2), J8.1 (Pin_1)
- net BOOT0: now also U1.44 (BOOT0)
- net BOOT1: now also J6.16 (Pin_16), U1.20 (PB2)
- net GND: now also J4.2 (Pin_2), J4.3 (Pin_3), J5.2 (Pin_2), J6.1 (Pin_1), J6.20 (Pin_20), J7.3 (Pin_3), J8.2 (Pin_2), J9.1 (Pin_1), U1.23 (VSS), U1.35 (VSS), U1.47 (VSS), U1.8 (VSSA)
- net RESET: now also J6.19 (Pin_19), U1.7 (NRST)
- net VBAT: now also J6.4 (Pin_4), U1.1 (VBAT)
- net at C3.2, Y1.1: now also U1.3 (PC14)
- net at C4.2, Y1.2: now also U1.4 (PC15)
- net at C7.2, R1.1, Y2.1: now also U1.6 (PD1)
- net at C8.2, R1.2, Y2.2: now also U1.5 (PD0)
- net PA4: now reaches J6.10 (Pin_10)
- net PA4: now also U1.14 (PA4)
- net PA5: now reaches J6.11 (Pin_11)
- net PA5: now also J4.7 (Pin_7), J5.3 (Pin_3), J8.7 (Pin_7), J9.3 (Pin_3), U1.15 (PA5), U1.16 (PA6)
- net PA6: now reaches J6.12 (Pin_12)
- net PA6: now also J8.9 (Pin_9), U1.17 (PA7)
- net PA7: now reaches J6.13 (Pin_13)
- net PA7: now also J4.8 (Pin_8), J5.4 (Pin_4), J8.6 (Pin_6), J9.4 (Pin_4), U1.29 (PA8)
- net PB0: now reaches J6.14 (Pin_14)
- net PB0: now also U1.18 (PB0)
- net PB1: now reaches J6.15 (Pin_15)
- net PB1: now also U1.19 (PB1)
- net PB10: now reaches J6.17 (Pin_17)
- net PB10: now also U1.21 (PB10)
- net PB11: now reaches J6.18 (Pin_18)
- net PB11: now also U1.22 (PB11)
- net LED2: now reaches J6.5 (Pin_5)
- net LED2: now also U1.2 (PC13)
- net PA0: now reaches J6.6 (Pin_6)
- net PA0: now also U1.10 (PA0)
- net PA1: now reaches J6.7 (Pin_7)
- net PA1: now also J8.14 (Pin_14), U1.11 (PA1)
- net PA2: now reaches J6.8 (Pin_8)
- net PA2: now also U1.12 (PA2)
- net PA3: now reaches J6.9 (Pin_9)
- net PA3: now also U1.13 (PA3)
- net PB3: now reaches J7.10 (Pin_10)
- net PB3: now also U1.39 (PB3)
- net PA15: now reaches J7.11 (Pin_11)
- net PA15: now also U1.38 (PA15)
- net PA12: now reaches J7.12 (Pin_12)
- net PA12: now also U1.33 (PA12)
- net PA11: now reaches J7.13 (Pin_13)
- net PA11: now also U1.32 (PA11)
- net PA10: now reaches J7.14 (Pin_14)
- net PA10: now also J8.11 (Pin_11)
- net PA9: now reaches J7.15 (Pin_15)
- net PA9: now also J8.12 (Pin_12), U1.31 (PA10)
- net PA8: now reaches J7.16 (Pin_16)
- net PA8: now also J8.13 (Pin_13), U1.30 (PA9)
- net PB15: now reaches J7.17 (Pin_17)
- net PB15: now also U1.28 (PB15)
- net PB14: now reaches J7.18 (Pin_18)
- net PB14: now also U1.27 (PB14)
- net PB13: now reaches J7.19 (Pin_19)
- net PB13: now also U1.26 (PB13)
- net PB12: now reaches J7.20 (Pin_20)
- net PB12: now also U1.25 (PB12)
- net PB9: now reaches J7.4 (Pin_4)
- net PB9: now also J4.11 (Pin_11), J8.3 (Pin_3), J9.7 (Pin_7), U1.46 (PB9)
- net PB8: now reaches J7.5 (Pin_5)
- net PB8: now also J4.10 (Pin_10), J8.4 (Pin_4), J9.5 (Pin_5), U1.45 (PB8)
- net PB7: now reaches J7.6 (Pin_6)
- net PB7: now also J4.9 (Pin_9), J8.5 (Pin_5), J9.6 (Pin_6), U1.43 (PB7)
- net PB6: now reaches J7.7 (Pin_7)
- net PB6: now also J4.6 (Pin_6), J8.8 (Pin_8), J9.8 (Pin_8), U1.42 (PB6)
- net PB5: now reaches J7.8 (Pin_8)
- net PB5: now also J8.10 (Pin_10), U1.41 (PB5)
- net PB4: now reaches J7.9 (Pin_9)
- net PB4: now also U1.40 (PB4)
- net SWCLK renamed PA14
- net PA14: now also U1.37 (PA14)
- net SWDAT renamed PA13
- net PA13: now also U1.34 (PA13)
- no-connect marks 0 -> 2
Other:
- moved on the sheet: C1, C10, C11, C12, C13, C14, C2, C3, C4, C5, C6, C7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

Commit message: update schematic diagram
Parts:
- J1: footprint Connector_USB:USB_Micro-AB_Molex_47590-0001 -> Connector_USB:USB_Micro-B_Molex-105017-0001
- J2: footprint Connector_PinSocket_2.54mm:PinSocket_1x06_P2.54mm_Vertical -> Connector_PinHeader_2.54mm:PinHeader_2x03_P2.54mm_Vertical
- SW1: footprint Button_Switch_THT:SW_MEC_5GTH9 -> Button_Switch_THT:SW_PUSH_6mm
- Y2: footprint Crystal:Crystal_HC49-U_Vertical -> Crystal:Crystal_HC18-U_Vertical
Changed lines of the file:
@@
 F 0 "Y2" V 7250 4150 50  0000 R CNN
 F 1 "8MHz" V 7300 4150 50  0000 R CNN
-F 2 "Crystal:Crystal_HC49-U_Vertical" H 7300 4300 50  0001 C CNN
+F 2 "Crystal:Crystal_HC18-U_Vertical" H 7300 4300 50  0001 C CNN
 F 3 "~" H 7300 4300 50  0001 C CNN
 	1    7300 4300
@@
 F 0 "J1" H 1900 2450 50  0000 C CNN
 F 1 "USB_B_Micro" H 1900 2350 50  0000 C CNN
-F 2 "Connector_USB:USB_Micro-AB_Molex_47590-0001" H 1950 1900 50  0001 C CNN
+F 2 "Connector_USB:USB_Micro-B_Molex-105017-0001" H 1950 1900 50  0001 C CNN
 F 3 "~" H 1950 1900 50  0001 C CNN
 	1    1800 1950
@@
 F 0 "J2" H 2600 5450 50  0000 C CNN
 F 1 "Conn_02x03_Odd_Even" H 2600 5000 50  0000 C CNN
-F 2 "Connector_PinSocket_2.54mm:PinSocket_1x06_P2.54mm_Vertical" H 2550 5250 50  0001 C CNN
+F 2 "Connector_PinHeader_2.54mm:PinHeader_2x03_P2.54mm_Vertical" H 2550 5250 50  0001 C CNN
 F 3 "~" H 2550 5250 50  0001 C CNN
 	1    2550 5250
@@
 F 0 "SW1" H 2950 8200 50  0000 C CNN
 F 1 "SW_Push" H 2950 8100 50  0000 C CNN
-F 2 "Button_Switch_THT:SW_MEC_5GTH9" H 2950 8100 50  0001 C CNN
+F 2 "Button_Switch_THT:SW_PUSH_6mm" H 2950 8100 50  0001 C CNN
 F 3 "~" H 2950 8100 50  0001 C CNN
 	1    2950 7900

Commit message: update
Parts:
- added P1: USB_C_Plug, Connector_USB:USB_C_Receptacle_Amphenol_12401610E4-2A, symbol Connector:USB_C_Plug
- added SW3: SW_Push, Button_Switch_THT:SW_PUSH-12mm, symbol Switch:SW_Push
- C11: value 104 -> 105
- Y1: footprint Crystal:Crystal_Round_D3.0mm_Vertical -> Crystal:Crystal_SMD_3215-2Pin_3.2x1.5mm
Connections:
- net PA0 is gone; now on net KEY0: J6.6 (Pin_6), U1.10 (PA0)
- net +5V: now also SW3.2; no longer J1.1 (VBUS), J8.1 (Pin_1)
- net GND: now also P1.A1 (GND), P1.A12 (GND), P1.B1 (GND), P1.B12 (GND), P1.S1 (SHIELD)
- net at J1.2 (D-), R5.2: now also P1.A7 (D-)
- net at J1.3 (D+), R3.2, R4.2: now also P1.A6 (D+)
- net +3V3 renamed +3.3V
- net +3.3V: now also J8.1 (Pin_1); no longer C11.2, C12.2, IC1.5 (VOUT)
- new net: C11.2, C12.2, IC1.5 (VOUT)
- new net: J1.1 (VBUS), P1.A4 (VBUS), P1.A9 (VBUS), P1.B4 (VBUS), P1.B9 (VBUS), SW3.1
- no-connect marks 2 -> 16
Other:
- moved on the sheet: C1, C10, C11, C12, C13, C2, C3, C4, C5, C6, C7, C8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
